File: RTCandIMU.kicad_sch (KiCad schematic)
At the start: 49 parts, among them Q2 NX3008NBKS, Q3 NX3008NBKS, Q4 MBT2222ADW1T1, Q5 MBT2222ADW1T1, Q6 NX3008NBKS, Q7 NX3008NBKS, Q8 MBT2222ADW1T1, Q9 MBT2222ADW1T1, U27 BNO085, U28 PCF8523TK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

Commit message: More stuff idk
Parts:
- added U34: INA219BxD, Package_SO:SOIC-8_3.9x4.9mm_P1.27mm, symbol Sensor_Energy:INA219BxD
Other:
- note added: "I2C Devices"
- note removed: "RTC and IMU"
