File: CM4_GPIO.kicad_sch (KiCad schematic)
At the start: 22 parts, among them J1 THD-20-R, J2 Micro_SD_Card, SW1 SW_DIP_x02, U1 TPD4EUSB30, U2 TPD4EUSB30, U3 74LVC1G07SE-7, U4 MagJack-A70-112-331N126

Commit message: More stuff idk
Parts:
- added R125: 0R (DNI), symbol Device:R_Small
- R2: value 0R (DNF) -> 0R (DNI)
Connections:
- net +3.3V: now also R125.1
- net GPIO_3.3V: now also R125.2
- net RF_DIO2 renamed GPIO26
- net RF_DIO3 renamed GPIO27
- net RF_DIO4 renamed GPIO2
- net RF_DIO5 renamed GPIO3
Other:
- note added: "NOTES: Potentially add SD load switch Decide whether to use 40-pin GPIO"
- note added: "Populate to use internal CM4 3.3V. Do not populate 3.3V regulator"
- moved on the sheet: D2, Module1A, R8
