File: CM4_HighSpeed.kicad_sch (KiCad schematic)
At the start: 4 parts, among them J3 Conn_01x22_Female, J4 Conn_01x22_Female, J5 690-019-298-412

Commit message: More stuff idk
Other:
- note added: "NOTES: Potentially add HDMI load switch Potentially add camera load switches"
- moved on the sheet: J5
