File: PiCubed.kicad_sch (KiCad schematic)
At the start: 53 parts

Commit message: Stash
Parts:
- removed C? (x2): 0.1uF, symbol Device:C_Small
- removed R? (x2): 2.2K, symbol Device:R_Small
- removed R?: 10K, symbol Device:R_Small
- removed U?: BMI260, Package_LGA:Bosch_LGA-14_3x2.5mm_P0.5mm, symbol Sensor_Motion:BMI160
- added C? (x3): 0.1uF, Capacitor_SMD:C_0603_1608Metric, symbol Device:C_Small
- added R? (x2): 10K, Resistor_SMD:R_0603_1608Metric, symbol Device:R_US
- added U?: BMX160, mainboard:BMX160, symbol mainboard:BMX160-symbols
- added U?: MAX706RESA+, Package_SO:SOIC-8_3.9x4.9mm_P1.27mm, symbol mainboard:MAX708RESA-T-symbols
Connections:
- net GND: now also C?.2, C?.2, C?.2, R?.1, U?.2 (GND_1), U?.3 (GND), U?.3 (GND_2), U?.4 (PFI), U?.6 (GNDIO), U?.7 (GND_3)
- net SCL_IMU: now also U?.13 (SCX)
- net SDA_IMU: now also U?.14 (SDX)
- new net: R?.2, U?.1 (SDO)
- new net: R?.2, U?.7 (~{RESET}), U?.8 (~{WDO})
- new net +3V3: C?.1, C?.1, C?.1, U?.12 (CSB), U?.2 (VCC), U?.5 (VDDIO), U?.8 (VDD)
- new net WDT_WDI: U?.6 (~{WDI})
- new net ~{RESET}: R?.1
- no-connect marks 50 -> 52
Other:
- note added: "0x68"
- note added: "I2C ADDR"
- note added: "WDT enabled when installed"
- moved on the sheet: C?, J?, R?, U?

Commit message: Update files to latest version
Parts:
- removed C?: 10uF, symbol Device:C_Small
- removed C? (x3): 0.1uF, Capacitor_SMD:C_0603_1608Metric, symbol Device:C_Small
- removed C? (x2): 100n, Capacitor_SMD:C_0402_1005Metric, symbol Device:C
- removed C?: 0.1uF, acheron_Components:C_0805_2012Metric, symbol Device:C_Small
- removed C? (x2): 10nF, Capacitor_SMD:C_0603_1608Metric, symbol Device:C
- removed C?: 0.1uF, Capacitor_SMD:C_0603_1608Metric, symbol mainboard:C_Small
- removed C?: 4.7nF, acheron_Components:C_0805_2012Metric, symbol Device:C_Small
- removed D?: WS2812B, LED_SMD:LED_WS2812B_PLCC4_5.0x5.0mm_P3.2mm, symbol LED:WS2812B
- removed J?: USB_C_Receptacle_USB2.0, symbol Connector:USB_C_Receptacle_USB2.0
- removed J? (x2): Conn_01x22, symbol Connector_Generic:Conn_01x22
- removed J?: Micro_SD_Card_Det, symbol Connector:Micro_SD_Card_Det
- removed J?: HDMI_C_1.4, symbol Connector:HDMI_C_1.4
- removed Module? (x2): ComputeModule4-CM4, CM4IO:Raspberry-Pi-4-Compute-Module, symbol CM4IO:ComputeModule4-CM4
- removed Q? (x4): BSS138DWQ-7, mainboard:BSS138DWQ-7, symbol mainboard:BSS138DWQ-7
- removed Q? (x4): MBT2222ADW1T1, Package_TO_SOT_SMD:SOT-363_SC-70-6, symbol Transistor_BJT:MBT2222ADW1T1
- removed R? (x2): 200K, Resistor_SMD:R_0603_1608Metric, symbol Device:R_US
- removed R? (x6): 10K, Resistor_SMD:R_0603_1608Metric, symbol Device:R_US
- removed R?: 0R, symbol Device:R_Small
- removed R? (x2): 680, Resistor_SMD:R_0603_1608Metric, symbol Device:R_US
- removed R?: 12K, symbol Device:R_Small
- removed R? (x2): 100K, Resistor_SMD:R_0603_1608Metric, symbol Device:R_US
- removed R? (x2): 5.1K, Resistor_SMD:R_0805_2012Metric_Pad1.20x1.40mm_HandSolder, symbol Device:R_Small
- removed R?: nF, symbol Device:R_Small
- removed R? (x2): 22, Resistor_SMD:R_0805_2012Metric_Pad1.20x1.40mm_HandSolder, symbol Device:R_Small
- removed R? (x2): 2.2K, symbol Device:R_Small
- removed R?: 1M, Resistor_SMD:R_0805_2012Metric_Pad1.20x1.40mm_HandSolder, symbol Device:R_Small
- removed U?: RT9742AGJ5F, Package_TO_SOT_SMD:TSOT-23-5, symbol Power_Management:RT9742AGJ5F
- removed U?: BMX160, mainboard:BMX160, symbol mainboard:BMX160-symbols
- removed U?: RT9742SNGV, Package_TO_SOT_SMD:SOT-23, symbol CM4IO:RT9742SNGV
- removed U?: MAX706RESA+, Package_SO:SOIC-8_3.9x4.9mm_P1.27mm, symbol mainboard:MAX708RESA-T-symbols
- removed U?: USBLC6-2SC6, Package_TO_SOT_SMD:SOT-23-6, symbol Power_Protection:USBLC6-2SC6
Connections:
- no-connect marks 52 -> 0
Other:
- added sheet Burn Wires (burnwires.kicad_sch)
- added sheet CM4_GPIO (CM4_GPIO.kicad_sch)
- added sheet CM4_HighSpeed (CM4_HighSpeed.kicad_sch)
- added sheet Connectors (connectors.kicad_sch)
- added sheet Payloads (payloads.kicad_sch)
- added sheet Power (power.kicad_sch)
- added sheet RTC and IMU (RTCandIMU.kicad_sch)
- added sheet Radio and GPS (radioandGPS.kicad_sch)
- added sheet USB-2 (USB-2.kicad_sch)
- added sheet USB-3 (USB-3.kicad_sch)
- note added: "Connectors ------- Ethernet SDCARD"
- note added: "Connectors ------- HDMI 0 CSI 0 CSI 1"
- note added: "Connectors ------- Quad USB 3.0"
- note added: "Connectors ------- Quad USB USB-C"
- note added: "PiCubed"
- note removed: "0x68"
- note removed: "I2C ADDR"
- note removed: "I2C Bus Protection - IMU"
- note removed: "Shield"
- note removed: "WDT enabled when installed"
- company: (none) -> RExLab Carnegie Mellon University
- title: (none) -> PiCubed Mainboard

Commit message: More stuff idk
Other:
- sheet RTC and IMU renamed I2C Devices
- added sheet Power2 (power2.kicad_sch)
- sheet CM4_GPIO ports: added none; removed RF_DIO2, RF_DIO3, RF_DIO4, RF_DIO5
- sheet I2C Devices: file RTCandIMU.kicad_sch -> I2CDevices.kicad_sch
- sheet I2C Devices ports: added BATT_SENSE_P; removed none
- sheet Radio and GPS ports: added none; removed RF_DIO2, RF_DIO3, RF_DIO4, RF_DIO5
- note added: "NOTES: FIX DNI LABELLING"

Commit message: Backup
Other:
- sheet Power2 renamed Power Regulation
- sheet Power Regulation: file power2.kicad_sch -> PowerRegulation.kicad_sch
Changed lines of the file:
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@@
 	(wire
 		(pts
-			(xy 142.621 154.94) (xy 154.94 154.94)
+			(xy 140.97 154.94) (xy 154.94 154.94)
 		)
 		(stroke
@@
 	(wire
 		(pts
-			(xy 142.621 152.4) (xy 154.94 152.4)
+			(xy 140.97 152.4) (xy 154.94 152.4)
 		)
 		(stroke
@@
 	(wire
 		(pts
-			(xy 142.621 149.86) (xy 154.94 149.86)
+			(xy 140.97 149.86) (xy 154.94 149.86)
 		)
 		(stroke
@@
 	)
 	(sheet
-		(at 96.52 143.51)
-		(size 46.101 16.383)
+		(at 95.25 142.24)
+		(size 45.72 17.653)
 		(stroke
 			(width 0.1524)
@@
 		)
 		(property "Sheetname" "Burn Wires"
-			(at 96.52 140.843 0)
+			(at 95.25 139.573 0)
 			(effects
 				(font
@@
 		)
 		(property "Sheetfile" "burnwires.kicad_sch"
-			(at 96.52 141.351 0)
+			(at 95.25 140.081 0)
 			(effects
 				(font
@@
 		)
 		(pin "BATT_P" input
-			(at 96.52 153.67 180)
+			(at 95.25 153.67 180)
 			(effects
 				(font
@@
 		)
 		(pin "RELAY_EN" input
-			(at 142.621 149.86 0)
+			(at 140.97 149.86 0)
 			(effects
 				(font
@@
 		)
 		(pin "BURN_PWM1" input
-			(at 142.621 154.94 0)
+			(at 140.97 154.94 0)
 			(effects
 				(font
@@
 		)
 		(pin "BURN_PWM0" input
-			(at 142.621 152.4 0)
+			(at 140.97 152.4 0)
 			(effects
 				(font
@@
 		)
 		(pin "VSOLAR" input
-			(at 96.52 149.86 180)
+			(at 95.25 149.86 180)
 			(effects
 				(font
@@
 	)
 	(sheet
-		(at 50.8 113.03)
-		(size 31.75 12.7)
+		(at 49.276 128.524)
+		(size 31.75 13.97)
 		(stroke
 			(width 0.1524)
@@
 		)
 		(property "Sheetname" "Power"
-			(at 50.8 110.363 0)
+			(at 49.276 125.857 0)
 			(effects
 				(font
@@
 		)
 		(property "Sheetfile" "power.kicad_sch"
-			(at 50.8 110.871 0)
+			(at 49.276 126.365 0)
 			(effects
 				(font
@@
 	)
 	(sheet
-		(at 51.816 136.525)
-		(size 31.877 12.065)
+		(at 50.8 105.41)
+		(size 31.75 13.97)
 		(stroke
 			(width 0.1524)
@@
 			(color 0 0 0 0.0000)
 		)
-		(property "Sheetname" "Power2"
-			(at 51.562 133.604 0)
+		(property "Sheetname" "Power Regulation"
+			(at 50.546 102.489 0)
 			(effects
 				(font
@@
 			)
 		)
-		(property "Sheetfile" "power2.kicad_sch"
-			(at 51.562 134.112 0)
-			(effects
-				(font
+		(property "Sheetfile" "PowerRegulation.kicad_sch"
+			(at 50.546 102.997 0)
+			(effects
+				(font
