File: USB-3.kicad_sch (KiCad schematic)
At the start: 89 parts, among them J10 USB3_A_Stacked, J9 USB3_A_Stacked, U14 UPD720201K8-711, U15 MR25H10CDF, U16 AP2191FMG-7, U17 AP2191FMG-7, U18 AP2191FMG-7, U19 AP2191FMG-7, U20 82401646, U21 82401646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

Commit message: More stuff idk
Other:
- note added: "NOTES: Add TPs for SPI ROM flash"
