File: radioandGPS.kicad_sch (KiCad schematic)
At the start: 18 parts, among them J11 Coax SMA, J12 Amphenol_901-144, J13 Amphenol_901-144, Q1 MMDT2907, U24 RFM98PW, U25 S1216V8, U26 EP2W+

Commit message: More stuff idk
Connections:
- net RF_DIO2: no longer names the net of U24.8 (GPIO_2)
- net RF_DIO3: no longer names the net of U24.3 (GPIO_3)
- net RF_DIO4: no longer names the net of U24.4 (GPIO_4)
- net RF_DIO5: no longer names the net of U24.15 (GPIO_5)
- no-connect marks 14 -> 18
